File: HARDWARE/iMX8MP-SOM-xGB-IND/Connectors.sch (KiCad schematic (older format))
At the start: 56 parts, among them Q2 Q32.768kHz/12.5pF/2P/SMD1206, Q3 Q24MHZ/20pF/20ppm/4P/3.2x2.5mm, T1 LMUN2235LT1G(SOT-23), T2 LMUN2235LT1G(SOT-23), T3 LMUN2235LT1G(SOT-23), U1 MIMX8ML8CVNKZAB(FCBGA548)

Commit message: Update
Parts:
- C120, C121, C122, C123, C124, C125: symbol OLIMEX_RCL:C -> iMX8MPLUS-SOM_Rev_B:C
- FET1, FET2, FET3, FET4, FET5, FET6: symbol OLIMEX_Transistors:N-MOS+DIOD -> iMX8MPLUS-SOM_Rev_B:N-MOS+DIOD
- GPIO1, GPIO2, GPIO3, GPIO5, GPIO6, LCD-LVDS1: symbol OLIMEX_Connectors:BH40S -> iMX8MPLUS-SOM_Rev_B:BH40S
- GPIO4: symbol OLIMEX_Connectors:BH20S -> iMX8MPLUS-SOM_Rev_B:BH20S
- MiPi_CSI1, MiPi_CSI2, MiPi_DSI1: symbol OLIMEX_Connectors:CON22 -> iMX8MPLUS-SOM_Rev_B:CON22
- Q2: symbol OLIMEX_Devices:Crystal -> iMX8MPLUS-SOM_Rev_B:Crystal
- Q3: symbol OLIMEX_Devices:Crystal_GND -> iMX8MPLUS-SOM_Rev_B:Crystal_GND
- R20, R21, R22, R23, R24, R25, R26, R27, R28, R29, R30, R31, R32, R33, R34, R35, R36, R37, R38, R39, R42, R43, R44, R45, R46, R47, R48: symbol OLIMEX_RCL:R -> iMX8MPLUS-SOM_Rev_B:R
- STAT_LED1: symbol OLIMEX_Diodes:LED -> iMX8MPLUS-SOM_Rev_B:LED
- T1, T2, T3: symbol OLIMEX_Transistors:LMUN2235LT1G(SOT-23) -> iMX8MPLUS-SOM_Rev_B:LMUN2235LT1G(SOT-23)
- U1: symbol OLIMEX_IC:MIMX8MP_BGA548 -> iMX8MPLUS-SOM_Rev_B:MIMX8MP_BGA548
