File: HARDWARE/iMX8MP-SOM-xGB-IND/Power Supply.sch (KiCad schematic (older format))
At the start: 123 parts, among them Q1 Q32.768kHz/12.5pF/2P/SMD1206, U1 MIMX8ML8CVNKZAB(FCBGA548), U2 PCA9450CHN(HVQFN56), U4 AT24C16C-SSHM-T(SOIC-8_150mil)

Commit message: Update
Parts:
- +5V0, GND1, NVCC_DRAM_1V1, NVCC_SD2, NVCC_SNVS_1V8, VDDA_1V8, VDD_1V8_1, VDD_3V3_1, VDD_ARM1, VDD_SOC1, VSD_3V3: symbol OLIMEX_OTHER:TESTPAD -> iMX8MPLUS-SOM_Rev_B:TESTPAD
- C100, C101, C102, C103, C104, C105, C106, C107, C108, C109, C110, C111, C112, C113, C114, C115, C116, C117, C118, C119, C26, C27, C28, C29, C30, C31, C32, C33, C34, C35, C36, C37, C38, C39, C40, C41, C42, C43, C44, C45, C46, C47, C48, C49, C50, C51, C52, C53, C54, C55, C56, C57, C58, C59, C60, C61, C62, C63, C64, C65, C66, C67, C68, C69, C70, C72, C74, C75, C76, C77, C78, C79, C80, C81, C82, C83, C84, C85, C86, C87, C89, C90, C91, C92, C93, C94, C95, C97, C98, C99: symbol OLIMEX_RCL:C -> iMX8MPLUS-SOM_Rev_B:C
- L1, L2, L3, L4, L5, L6: symbol OLIMEX_RCL:L -> iMX8MPLUS-SOM_Rev_B:L
- Q1: symbol OLIMEX_Devices:Crystal -> iMX8MPLUS-SOM_Rev_B:Crystal
- R11, R12, R13, R14, R15, R16, R17, R18, R19, R40, R41: symbol OLIMEX_RCL:R -> iMX8MPLUS-SOM_Rev_B:R
- U1: symbol OLIMEX_IC:MIMX8MP_BGA548 -> iMX8MPLUS-SOM_Rev_B:MIMX8MP_BGA548
- U2: symbol OLIMEX_IC:PCA9450 -> iMX8MPLUS-SOM_Rev_B:PCA9450
- U4: symbol OLIMEX_IC:AT24C16BN-SH(SO-8_150mil) -> iMX8MPLUS-SOM_Rev_B:AT24C16BN-SH(SO-8_150mil)
