File: HARDWARE/iMX8MP-SOM-xGB-IND/iMX8MPLUS-SOM_Rev_B.sch (KiCad schematic (older format))
At the start: 47 parts, among them IC1 K4F6E304HB-MGCJ, U1 MIMX8ML8CVNKZAB(FCBGA548)

Commit message: Update
Parts:
- C1, C10, C11, C12, C13, C14, C15, C16, C17, C18, C19, C2, C20, C21, C22, C23, C24, C25, C3, C4, C5, C6, C7, C8, C9: symbol OLIMEX_RCL:C -> iMX8MPLUS-SOM_Rev_B:C
- FID1, FID2, FID3, FID4, FID5, FID6: symbol OLIMEX_OTHER:Fiducial -> iMX8MPLUS-SOM_Rev_B:Fiducial
- IC1: symbol OLIMEX_IC:MT53B768M32D4NQ_200P -> iMX8MPLUS-SOM_Rev_B:MT53B768M32D4NQ_200P
- MH1, MH2, MH3, MH4: symbol OLIMEX_OTHER:Mounting_Hole_NPTH -> iMX8MPLUS-SOM_Rev_B:Mounting_Hole_NPTH
- R1, R10, R2, R3, R4, R5, R6, R7, R8, R9: symbol OLIMEX_RCL:R -> iMX8MPLUS-SOM_Rev_B:R
- U1: symbol OLIMEX_IC:MIMX8MP_BGA548 -> iMX8MPLUS-SOM_Rev_B:MIMX8MP_BGA548
